File: floppapad2.kicad_sch (KiCad schematic)
At the start: 41 parts, among them J1 USBC, J2 DBG, SW1 SW_Push, SW10 SW_Push, SW11 RotaryEncoder_Switch, SW12 BOOT, SW2 SW_Push, SW3 SW_Push, SW4 SW_Push, SW5 SW_Push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

Commit message: slight adjustment
Changed lines of the file:
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@@
       (effects (font (size 1.27 1.27)))
     )
-    (property "Value" "100n" (at 90.17 27.94 0)
+    (property "Value" "100n" (at 97.79 27.94 0)
       (effects (font (size 1.27 1.27)))
     )
@@
   (symbol (lib_id "Device:C_Small") (at 93.98 26.67 0) (mirror x) (unit 1)
     (in_bom yes) (on_board yes) (dnp no)
-    (property "Reference" "C8" (at 91.44 25.4 0)
+    (property "Reference" "C8" (at 96.52 25.4 0)
       (effects (font (size 1.27 1.27)))
     )

Commit message: better debug
Parts:
- J2: footprint Connector_PinSocket_2.54mm:PinSocket_1x04_P2.54mm_Vertical -> Connector_PinSocket_2.54mm:PinSocket_1x03_P2.54mm_Vertical; symbol Connector_Generic:Conn_01x04 -> Connector_Generic:Conn_01x03
Connections:
- net +3.3V: no longer J2.4 (Pin_4)
Changed lines of the file:
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@@
-    )
-  )
-  (symbol (lib_id "power:+3.3V") (at 189.23 120.015 0) (unit 1)
-    (in_bom yes) (on_board yes) (dnp no)
-    (property "Reference" "#PWR039" (at 189.23 123.825 0)
-      (effects (font (size 1.27 1.27)) hide)
-    )
-    (property "Value" "+3.3V" (at 189.23 116.205 0)
-      (effects (font (size 1.27 1.27)))
-    )
-    (property "Footprint" "" (at 189.23 120.015 0)
-      (effects (font (size 1.27 1.27)) hide)
-    )
-    (property "Datasheet" "" (at 189.23 120.015 0)
-      (effects (font (size 1.27 1.27)) hide)
-    )
-    (pin "1")
-    (instances
-      (project "floppapad2"
-        (path "/5135f742-4682-42d0-97bb-739add528f37"
-          (reference "#PWR039") (unit 1)
-        )
-      )
     )
   )
@@
     )
   )
-  (symbol (lib_id "Connector_Generic:Conn_01x04") (at 184.15 125.095 180) (unit 1)
+  (symbol (lib_id "Connector_Generic:Conn_01x03") (at 184.15 125.095 180) (unit 1)
     (in_bom yes) (on_board yes) (dnp no) (fields_autoplaced)
-    (property "Reference" "J2" (at 184.15 114.3 0)
-      (effects (font (size 1.27 1.27)))
-    )
-    (property "Value" "DBG" (at 184.15 116.84 0)
-      (effects (font (size 1.27 1.27)))
-    )
-    (property "Footprint" "Connector_PinSocket_2.54mm:PinSocket_1x04_P2.54mm_Vertical" (at 184.15 125.095 0)
+    (property "Reference" "J2" (at 184.15 116.84 0)
+      (effects (font (size 1.27 1.27)))
+    )
+    (property "Value" "DBG" (at 184.15 119.38 0)
+      (effects (font (size 1.27 1.27)))
+    )
+    (property "Footprint" "Connector_PinSocket_2.54mm:PinSocket_1x03_P2.54mm_Vertical" (at 184.15 125.095 0)
       (effects (font (size 1.27 1.27)) hide)
     )
@@
     (pin "2")
     (pin "3")
-    (pin "4")
-    (instances
-      (project "floppapad2"
+    (instances
+      (project "floppapad2"
